Commit message: created custom ros2 package

File: nautilus_ws/src/nautilus_bringup/nautilus_auv/BlueRov2.urdf (robot description, URDF)
Before this commit: robot BlueRov2, 22 links, 21 joints
Links:
- link base_link: mass 100 -> 7

File: nautilus_ws/src/nautilus_bringup/nautilus_auv/BlueRov2.urdf.xacro (robot description, xacro)
@@ -1,9 +1,9 @@
 <?xml version='2.0'?>
 <robot xmlns:xacro="http://www.ros.org/wiki/xacro" name="BlueRov2">
-    <xacro:include filename="../Part/Thruster/T200.urdf.xacro" />
-    <xacro:include filename="../Part/IMU/IMU.urdf.xacro" />
-    <xacro:include filename="../Part/Camera/Camera.urdf.xacro" />
-    <xacro:include filename="../Part/Camera/CameraDepth.urdf.xacro" />
-    <xacro:include filename="../Part/Camera/CameraStereo.urdf.xacro" />
+    <xacro:include filename="./Part/Thruster/T200.urdf.xacro" />
+    <xacro:include filename="./Part/IMU/IMU.urdf.xacro" />
+    <xacro:include filename="./Part/Camera/Camera.urdf.xacro" />
+    <xacro:include filename="./Part/Camera/CameraDepth.urdf.xacro" />
+    <xacro:include filename="./Part/Camera/CameraStereo.urdf.xacro" />
     <link name="base_link">
         <visual>
@@ -16,5 +16,5 @@
         <inertial>
         <origin xyz="0 0 0" rpy="0 0 0"/>
-        <mass value="100"/>
+        <mass value="7"/>
         <inertia
         ixx="1"
@@ -136,32 +136,28 @@
             </control>
         </plugin>
-    </gazebo>
-    <gazebo>
-        <!-- buoyancy plugin -->
-        <plugin name="ignititon::gazebo::systems::Buoyancy" filename="ignition-gazebo-buoyancy-system">
-            <!-- <descriptionParam>robot_description</descriptionParam>
-            <fluidTopic>current</fluidTopic>
-            <alwaysOn>true</alwaysOn>
-            <surface>0 0 0</surface>
-            <updateRate>.001</updateRate>
-            <link name="base_link">
-                <buoyancy>
-                <compensation>0.2525</compensation>
-                <origin xyz= "0.12585 0.111 0.1789"/>
-                </buoyancy>
-                <buoyancy>
-                <compensation>0.2525</compensation>
-                <origin xyz= "-0.12585 0.111 0.1789"/>
-                </buoyancy>
-                <buoyancy>
-                <compensation>0.2525</compensation>
-                <origin xyz= "-0.12585 -0.111 0.1789"/>
-                </buoyancy>
-                <buoyancy>
-                <compensation>0.2525</compensation>
-                <origin xyz= "0.12585 -0.111 0.1789"/>
-                </buoyancy>
-            </link> -->
-        </plugin>
+<!--
+        <plugin
+        filename="gz-sim-hydrodynamics-system"
+        name="gz::sim::systems::Hydrodynamics">
+            <link_name>base_link</link_name>
+            <xDotU>-4.876161</xDotU>
+            <yDotV>-126.324739</yDotV>
+            <zDotW>-126.324739</zDotW>
+            <kDotP>0</kDotP>
+            <mDotQ>-33.46</mDotQ>
+            <nDotR>-33.46</nDotR>
+            <xUabsU>-6.2282</xUabsU>
+            <xU>0</xU>
+            <yVabsV>-601.27</yVabsV>
+            <yV>0</yV>
+            <zWabsW>-601.27</zWabsW>
+            <zW>0</zW>
+            <kPabsP>-0.1916</kPabsP>
+            <kP>0</kP>
+            <mQabsQ>-632.698957</mQabsQ>
+            <mQ>0</mQ>
+            <nRabsR>-632.698957</nRabsR>
+            <nR>0</nR>
+        </plugin> -->
     </gazebo>
 </robot>

Commit message: added hydrodynamics plugin, values are not necessarily realistic but are functional for now

File: nautilus_ws/src/nautilus_bringup/nautilus_auv/BlueRov2.urdf (robot description, URDF)
Before this commit: robot BlueRov2, 22 links, 21 joints
Links:
- link base_link: mass 7 -> 8

File: nautilus_ws/src/nautilus_bringup/nautilus_auv/BlueRov2.urdf.xacro (robot description, xacro)
@@ -15,6 +15,6 @@
         </visual>
         <inertial>
-        <origin xyz="0 0 0" rpy="0 0 0"/>
-        <mass value="7"/>
+        <origin xyz="0 0 -0.1" rpy="0 0 0"/>
+        <mass value="8"/>
         <inertia
         ixx="1"
@@ -136,28 +136,27 @@
             </control>
         </plugin>
-<!--
         <plugin
-        filename="gz-sim-hydrodynamics-system"
-        name="gz::sim::systems::Hydrodynamics">
+            filename="gz-sim-hydrodynamics-system"
+            name="gz::sim::systems::Hydrodynamics">
             <link_name>base_link</link_name>
-            <xDotU>-4.876161</xDotU>
-            <yDotV>-126.324739</yDotV>
-            <zDotW>-126.324739</zDotW>
-            <kDotP>0</kDotP>
-            <mDotQ>-33.46</mDotQ>
-            <nDotR>-33.46</nDotR>
-            <xUabsU>-6.2282</xUabsU>
-            <xU>0</xU>
-            <yVabsV>-601.27</yVabsV>
-            <yV>0</yV>
-            <zWabsW>-601.27</zWabsW>
-            <zW>0</zW>
-            <kPabsP>-0.1916</kPabsP>
-            <kP>0</kP>
-            <mQabsQ>-632.698957</mQabsQ>
-            <mQ>0</mQ>
-            <nRabsR>-632.698957</nRabsR>
-            <nR>0</nR>
-        </plugin> -->
+            <xDotU>1</xDotU>
+            <yDotV>1</yDotV>
+            <zDotW>2.5</zDotW>
+            <kDotP>0.075</kDotP>
+            <mDotQ>0.075</mDotQ>
+            <nDotR>0.135</nDotR>
+            <xUabsU>-20</xUabsU>
+            <xU>-5</xU>
+            <yVabsV>-20</yVabsV>
+            <yV>-5</yV>
+            <zWabsW>-50</zWabsW>
+            <zW>-5</zW>
+            <kPabsP>-0.5</kPabsP>
+            <kP>-0.05</kP>
+            <mQabsQ>-0.5</mQabsQ>
+            <mQ>-0.05</mQ>
+            <nRabsR>-1</nRabsR>
+            <nR>-0.1</nR>
+        </plugin>
     </gazebo>
 </robot>

Commit message: Added lift drag to thrusters in order to produce thrust

File: nautilus_ws/src/nautilus_bringup/nautilus_auv/BlueRov2.urdf (robot description, URDF)
Before this commit: robot BlueRov2, 22 links, 21 joints
Links:
- link base_link: mass 8 -> 9

File: nautilus_ws/src/nautilus_bringup/nautilus_auv/BlueRov2.urdf.xacro (robot description, xacro)
@@ -16,5 +16,5 @@
         <inertial>
         <origin xyz="0 0 -0.1" rpy="0 0 0"/>
-        <mass value="8"/>
+        <mass value="9"/>
         <inertia
         ixx="1"

File: nautilus_ws/src/nautilus_bringup/nautilus_auv/Part/Thruster/T200.urdf.xacro (robot description, xacro)
@@ -81,5 +81,5 @@
     </joint>
     <gazebo>
-      <!--plugin name="${name}_propeller_plugin" filename="libLiftDragPlugin.so">
+      <plugin name="gz::sim::systems::LiftDrag" filename="gz-sim-lift-drag-system">
         <a0>0.3</a0>
         <alpha_stall>1.4</alpha_stall>
@@ -96,5 +96,5 @@
         <upward>0 0 -1</upward>
         <link_name>${name}_propeler</link_name>
-      </plugin-->
+      </plugin>
     </gazebo>
   </xacro:macro>
