Commit message: NSFW-36 Saving current progress on gazebo simulator

File: nautilus_ws/src/nautilus_bringup/nautilus_auv/BlueRov2.urdf.xacro (robot description, xacro)
@@ -6,4 +6,6 @@
     <xacro:include filename="./Part/Camera/CameraDepth.urdf.xacro" />
     <xacro:include filename="./Part/Camera/CameraStereo.urdf.xacro" />
+    <xacro:include filename="./Part/DVL/DVL.urdf.xacro" />
+    <xacro:include filename="./Part/DepthSensor/DepthSensor.urdf.xacro"/>
     <link name="base_link">
         <visual>
@@ -36,4 +38,13 @@
     <xacro:CameraDepth name="camera" link="base_link" xyz="0.2 0 0" rpy="0 0 0" />
     <!--<xacro:CameraStero name="camera_stereo" link="base_link" xyz="0.2 0 0" rpy="0 0 0" />-->
+    <xacro:dvl_sensor name="dvl_front"
+                  parent_link="base_link"
+                  update_rate="10"
+                  aperture="3.0" tilt="30.0"
+                  min_range="0.3" max_range="40.0" resolution="0.01"
+                  ref_frame="parent"
+                  bottom_stddev="0.01"
+                  wm_enabled="true" wm_bins="10" wm_near="20.0" wm_far="60.0" wm_stddev="0.05"/>
+	<xacro:DepthSensor parent_link="base_link" sensor_name="water_pressure"/>
     <xacro:T200 name="thruster1" fixTo="base_link" xyz="0.125 -0.105 0.02" RPY="1.5707963 1.5707963 -0.78539815"/>
     <xacro:T200 name="thruster2" fixTo="base_link" xyz="0.125 0.105 0.02" RPY="1.5707963 1.5707963 3.92699075"/>
@@ -135,4 +146,8 @@
             <multiplier>102</multiplier>
             </control>
+            <barometer>
+            	<name>water_pressure</name>
+            	<linkName>base_link</linkName>
+            </barometer>
         </plugin>
         <plugin

File: nautilus_ws/src/nautilus_bringup/nautilus_auv/Part/DVL/DVL.urdf.xacro (robot description, xacro)
@@ -1,21 +1,47 @@
-<?xml version='1.0'?>
-<robot xmlns:xacro="http://www.ros.org/wiki/xacro" name="DVL">
-  <xacro:macro name="DVL" params="link topicName noise Hz">
-    <gazebo>
-        <plugin name="gazebo_ros_DVL" filename="libgazebo_ros_DVL.so">
-            <ros>
-                <!-- Add a namespace -->
-                <namespace>/DVL</namespace>
-                <!-- Remap the default topic -->
-                <remapping>odom:=${topicName}</remapping>
-            </ros>
-            <!-- Name of the link within this model whose pose will be published -->
-            <body_name>${link}</body_name>
-            <!-- Update rate in Hz, defaults to 0.0, which means as fast as possible -->
-            <update_rate>${Hz}</update_rate>
-            <!-- Standard deviation of the noise to be added to the reported velocities. -->
-            <gaussian_noise>${noise}</gaussian_noise>
-        </plugin>
-    </gazebo>
+<?xml version="1.0"?>
+<sdf version="1.10" xmlns:xacro="http://www.ros.org/wiki/xacro" xmlns:gz="http://gazebosim.org/schema">
+  <xacro:macro name="dvl_sensor"
+               params="name parent_link:=base_link update_rate:=10
+                       aperture:=3.0 tilt:=30.0 degrees:=true
+                       min_range:=0.3 max_range:=40.0 resolution:=0.01
+                       ref_frame:=parent bottom_stddev:=0.01 bottom_visualize:=false
+                       wm_enabled:=true wm_bins:=10 wm_near:=20.0 wm_far:=60.0 wm_stddev:=0.05 wm_visualize:=false">
+    <model name="${name}_model">
+      <link name="${parent_link}">
+        <sensor name="${name}" type="custom" gz:type="dvl">
+          <update_rate>${update_rate}</update_rate>
+          <gz:dvl>
+            <arrangement degrees="${degrees}">
+              <beam id="1"><aperture>${aperture}</aperture><rotation>45</rotation><tilt>${tilt}</tilt></beam>
+              <beam id="2"><aperture>${aperture}</aperture><rotation>-45</rotation><tilt>${tilt}</tilt></beam>
+              <beam id="3"><aperture>${aperture}</aperture><rotation>135</rotation><tilt>${tilt}</tilt></beam>
+              <beam id="4"><aperture>${aperture}</aperture><rotation>-135</rotation><tilt>${tilt}</tilt></beam>
+            </arrangement>
+            <tracking>
+              <bottom_mode>
+                <noise type="gaussian"><stddev>${bottom_stddev}</stddev></noise>
+                <visualize>${bottom_visualize}</visualize>
+              </bottom_mode>
+              <water_mass_mode>
+                <when>${wm_enabled}</when>
+                <water_velocity><x>0</x><y>0</y><z>0</z></water_velocity>
+                <boundaries><near>${wm_near}</near><far>${wm_far}</far></boundaries>
+                <bins>${wm_bins}</bins>
+                <noise type="gaussian"><stddev>${wm_stddev}</stddev></noise>
+                <visualize>${wm_visualize}</visualize>
+              </water_mass_mode>
+            </tracking>
+            <minimum_range>${min_range}</minimum_range>
+            <maximum_range>${max_range}</maximum_range>
+            <resolution>${resolution}</resolution>
+            <reference_frame>${ref_frame}</reference_frame>
+          </gz:dvl>
+          <plugin
+            filename="tethys-dopplervelocitylogsystem"
+            name="tethys::DopplerVelocityLogSystem">
+          </plugin>
+        </sensor>
+      </link>
+    </model>
   </xacro:macro>
-</robot>
+</sdf>

File: nautilus_ws/src/nautilus_bringup/nautilus_auv/Part/DepthSensor/DepthSensor.urdf.xacro (robot description, xacro)
@@ -1,21 +1,12 @@
 <?xml version='1.0'?>
 <robot xmlns:xacro="http://www.ros.org/wiki/xacro" name="DepthSensor">
-  <xacro:macro name="DepthSensor" params="link topicName sealevel noise Hz">
-    <gazebo>
-        <plugin name="gazebo_ros_DepthSensor" filename="libgazebo_ros_DepthSensor.so">
-            <ros>
-                <!-- Add a namespace -->
-                <namespace>/depthSensor</namespace>
-                <!-- Remap the default topic -->
-                <remapping>odom:=${topicName}</remapping>
-            </ros>
-            <!-- Name of the link within this model whose pose will be published -->
-            <body_name>${link}</body_name>
-            <!-- Update rate in Hz, defaults to 0.0, which means as fast as possible -->
-            <update_rate>${Hz}</update_rate>
-            <sea_level>${sealevel}</sea_level>
-            <!-- Standard deviation of the noise to be added to the reported velocities. -->
-            <gaussian_noise>${noise}</gaussian_noise>
-        </plugin>
+  <xacro:macro name="DepthSensor" params="parent_link sensor_name">
+    <gazebo reference="${parent_link}">
+      <sensor name="${sensor_name}" type="air_pressure">
+        <always_on>true</always_on>
+        <update_rate>50</update_rate>
+        <pose>0 0 0 0 0 0</pose>
+        <topic>/${sensor_name}</topic>
+      </sensor>
     </gazebo>
   </xacro:macro>

File: nautilus_ws/src/nautilus_bringup/nautilus_auv/Part/IMU/IMU.urdf.xacro (robot description, xacro)
@@ -71,10 +71,7 @@
                 </linear_acceleration>
             </imu>
-            <plugin name="bytes_imu" filename="libgazebo_ros_imu_sensor.so">
-                <ros>
-                    <namespace>imu</namespace>
-                    <remapping>~/out:=data_raw</remapping>
-                </ros>
-                <initial_orientation_as_reference>false</initial_orientation_as_reference>
+            <plugin
+                filename="gz-sim-imu-system"
+                name="gz::sim::systems::Imu">
             </plugin>
         </sensor>

File: nautilus_ws/src/nautilus_bringup/nautilus_auv/Part/Thruster/T200.urdf.xacro (robot description, xacro)
@@ -58,4 +58,9 @@
           <box size="0.0225 0.01  0.005"/>
         </geometry>
+        <!-- <material>
+          <ambient>1 0 0 1</ambient>
+          <diffuse>1 0 0 1</diffuse>
+          <specular>0.1 0.1 0.1 1</specular>
+        </material> -->
       </visual>
       <visual name="blade2">
@@ -64,4 +69,10 @@
           <box size="0.0225 0.01  0.005"/>
         </geometry>
+        <!-- <material>
+          <ambient>1.0 0.0 0.0 1.0</ambient>
+          <diffuse>1.0 0.0 0.0 1.0</diffuse>
+          <specular>1.0 0.0 0.0 1.0</specular>
+          <emissive>1.0 0.0 0.0 1.0</emissive>
+        </material> -->
       </visual>
       <!--<visual name='${name}_propeler_visual'>
@@ -94,4 +105,20 @@
         <cp>-0.084 0 0</cp>
         <forward>0 -1 0</forward>
+        <upward>0 0 1</upward>
+        <link_name>${name}_propeler</link_name>
+      </plugin>
+      <plugin name="gz::sim::systems::LiftDrag" filename="gz-sim-lift-drag-system">
+        <a0>0.3</a0>
+        <alpha_stall>1.4</alpha_stall>
+        <cla>4.2500</cla>
+        <cda>0.10</cda>
+        <cma>0.00</cma>
+        <cla_stall>-0.025</cla_stall>
+        <cda_stall>0.0</cda_stall>
+        <cma_stall>0.0</cma_stall>
+        <area>0.002</area>
+        <air_density>1000</air_density>
+        <cp>-0.084 0 0</cp>
+        <forward>0 1 0</forward>
         <upward>0 0 -1</upward>
         <link_name>${name}_propeler</link_name>

Commit message: NSFW-85 saved emiles progress

File: nautilus_ws/src/nautilus_bringup/nautilus_auv/BlueRov2.urdf.xacro (robot description, xacro)
@@ -37,5 +37,6 @@
     <!--<xacro:Camera name="camera_front" link="base_link" xyz="0.2 0 0" rpy="0 0 0" />-->
     <xacro:Camera name="camera" link="base_link" xyz="0.2 0 0" rpy="0 0 0" />
-    <!--<xacro:CameraStero name="camera_stereo" link="base_link" xyz="0.2 0 0" rpy="0 0 0" />-->
+    <xacro:CameraDepth name="cameraDepth" link="base_link" xyz="0.2 0 0" rpy="0 0 0" />
+    <!-- <xacro:CameraStero name="camera_stereo" link="base_link" xyz="0.2 0 0" rpy="0 0 0" /> -->
     <xacro:dvl_sensor name="dvl_front"
                   parent_link="base_link"

File: nautilus_ws/src/nautilus_bringup/nautilus_auv/Part/Camera/CameraDepth.urdf.xacro (robot description, xacro)
@@ -1,6 +1,10 @@
 <?xml version='1.0'?>
-<robot xmlns:xacro="http://www.ros.org/wiki/xacro" name="CameraDepth">
+<robot xmlns:xacro="http://www.ros.org/wiki/xacro" name="Camera">
   <xacro:macro name="CameraDepth" params="name link xyz rpy">
-    <link name="${name}_link">
+    <!--    set property   -->
+    <xacro:property name="xyzFrameCam" value="0 0 0" />
+    <xacro:property name="rpyFrameCam" value="0 0 0" />
+    <!--    define link  -->
+    <link name="${name}_camera_link">
         <visual>
             <geometry>
@@ -9,29 +13,54 @@
         </visual>
         <inertial>
-            <origin xyz="0 0.069 -0.047" rpy="0 0 0"/>
-            <mass value="0.0001"/>
+            <origin xyz="0 0 0" rpy="0 0 0"/>
+            <mass value="0.0035"/>
             <inertia
-                ixx="1"
-                ixy="0"
-                ixz="0"
-                iyy="1"
-                iyz="0"
-                izz="1"/>
+            ixx="1"
+            ixy="0"
+            ixz="0"
+            iyy="1"
+            iyz="0"
+            izz="1"/>
         </inertial>
     </link>
-    <gazebo reference="${name}_link">
+    <gazebo reference="${name}_camera_link">
         <material>Gazebo/Black</material>
     </gazebo>
-    <joint name="${name}_joint" type="fixed">
+    <joint name="${name}_camera_joint" type="fixed">
         <parent link="${link}"/>
-        <child link="${name}_link"/>
+        <child link="${name}_camera_link"/>
         <origin rpy="${rpy}" xyz="${xyz}"/>
-        <axis xyz="0 0 1" />
+        <axis xyz="1 0 0" />
     </joint>
-    <gazebo reference="${name}_joint">
+    <gazebo reference="${name}_camera_joint">
         <preserveFixedJoint>true</preserveFixedJoint>
-        <material>Gazebo/Black</material>
     </gazebo>
-    <link name="${name}_rgb_optical_frame">
+    <link name="${name}_camera_frame">
+        <visual>
+            <geometry>
+                <box size="0.005 0.01 0.01"/>
+            </geometry>
+        </visual>
+        <inertial>
+            <origin xyz="0 0 0" rpy="0 0 0"/>
+            <mass value="0.0035"/>
+            <inertia
+            ixx="1"
+            ixy="0"
+            ixz="0"
+            iyy="1"
+            iyz="0"
+            izz="1"/>
+        </inertial>
+    </link>
+    <joint name="${name}_camera_frame_joint" type="fixed">
+        <parent link="${name}_camera_link"/>
+        <child link="${name}_camera_frame"/>
+        <origin rpy="${rpyFrameCam}" xyz="${xyzFrameCam}"/>
+    </joint>
+    <gazebo reference="${name}_camera_frame_joint">
+        <preserveFixedJoint>true</preserveFixedJoint>
+    </gazebo>
+    <link name="${name}_camera_depth_optical_frame">
         <inertial>
             <origin xyz="0 0.069 -0.047" rpy="0 0 0"/>
@@ -46,53 +75,68 @@
         </inertial>
     </link>
-    <joint name="${name}_rgb_optical_joint" type="fixed">
-            <parent link="${name}_link"/>
-            <child link="${name}_rgb_optical_frame"/>
+    <joint name="${name}_camera_depth_optical_joint" type="fixed">
+            <parent link="${name}_camera_frame"/>
+            <child link="${name}_camera_depth_optical_frame"/>
             <origin rpy="${-pi/2} 0 ${-pi/2}" xyz="0 0 0"/>
             <axis xyz="0 0 1" />
     </joint>
-    <gazebo reference="${name}_rgb_optical_joint">
+    <gazebo reference="${name}_camera_depth_optical_joint">
         <preserveFixedJoint>true</preserveFixedJoint>
     </gazebo>
     <!-- camera -->
-    <gazebo reference="${name}_link">
-            <sensor name="${name}" type="depth">
-                <!--<frameName>${name}_rgb_optical_frame</frameName>-->
-                <always_on>true</always_on>
+    <gazebo reference="${name}_camera_frame">
+        <sensor type="depth_camera" name="${name}_depth_sensor">
+        <always_on>true</always_on>
+        <visualize>true</visualize>
+        <update_rate>10.0</update_rate>
+        <topic>camera/depth/image_raw</topic>
+        <gz_frame_id>camera_depth_frame</gz_frame_id>
+        <camera name="head">
+        <!-- https://elinux.com/Rpi_Camera_Module  -->
+            <horizontal_fov>1.0855</horizontal_fov>
+            <!-- vertical_fov>0.85169</vertical_fov -->
+            <image>
+            <width>1920</width>
+            <height>1080</height>
+            <format>B8G8R8</format>
+            </image>
+            <clip>
+            <near>0.01</near>
+            <far>500</far>
+            </clip>
+            <min_depth>0.1</min_depth>
+            <max_depth>50.0</max_depth>
+            <noise>
+            <type>gaussian</type>
+            <!-- Noise is sampled independently per pixel on each frame.
+                That pixel's noise value is added to each of its color
+                channels, which at that point lie in the range [0,1]. -->
+            <mean>0.0</mean>
+            <stddev>0.007</stddev>
+            </noise>
+        </camera>
+        <depth_camera>
+        <clip>
+          <near>0.1</near>
+          <far>50.0</far>
+        </clip>
+      </depth_camera>
+            <!-- <plugin name="camera_controller" filename="libgazebo_ros_camera.so">
+            <frame_name>${name}_camera_rgb_optical_frame</frame_name>
+                <alwaysOn>true</alwaysOn>
                 <visualize>true</visualize>
-                <update_rate>30</update_rate>
-                <camera name="intel_realsense_r200">
-                <horizontal_fov>1.02974</horizontal_fov>
-                <image>
-                    <width>640</width>
-                    <height>480</height>
-                    <format>R8G8B8</format>
-                </image>
-                <clip>
-                    <near>0.05</near>
-                    <far>50</far>
-                </clip>
-                <noise>
-                    <type>gaussian</type>
-                    <!-- Noise is sampled independently per pixel on each frame.
-                        That pixel's noise value is added to each of its color
-                        channels, which at that point lie in the range [0,1]. -->
-                    <mean>0.0</mean>
-                    <stddev>0.007</stddev>
-                </noise>
-                </camera>
-                <plugin name="camera_driver" filename="libgazebo_ros_camera.so">
-                    <camera_name>${name}</camera_name>
-                    <frame_name>${name}_rgb_optical_frame</frame_name>
-                    <ros>
-                    <!-- <namespace>test_cam</namespace> -->
-                    <!-- <remapping>image_raw:=image_demo</remapping> -->
-                    <!-- <remapping>camera_info:=camera_info_demo</remapping> -->
-                    </ros>
-                    <!-- camera_name>omit so it defaults to sensor name</camera_name-->
-                    <!-- frame_name>omit so it defaults to link name</frameName-->
-                    <!-- <hack_baseline>0.07</hack_baseline> -->
-                </plugin>
-            </sensor>
+                <updateRate>30.0</updateRate>
+                <cameraName>camera</cameraName>
+                <imageTopicName>image_raw</imageTopicName>
+                <cameraInfoTopicName>camera_info</cameraInfoTopicName>
+                <frame_Name>${name}_camera_frame_joint</frame_Name>
+                <hackBaseline>0.07</hackBaseline>
+                <distortionK1>0.0</distortionK1>
+                <distortionK2>0.0</distortionK2>
+                <distortionK3>0.0</distortionK3>
+                <distortionT1>0.0</distortionT1>
+                <distortionT2>0.0</distortionT2>
+            </plugin> -->
+        </sensor>
     </gazebo>
   </xacro:macro>
